File: Two Nine Five/Two Nine Five Rev 2.brd (EAGLE design)
At the start: 68 x 106 mm, 175 parts, among them U16 TL072, U2 TL072, U3 TL074, U4 TL074, U5 TL072

Commit message: Change R34 from 15k to 18k on all schematics
Parts:
- R34: value 15k -> 18k
